File: KiCAD/NewsBox_V1/NewsBox.kicad_pcb (KiCad board)
At the start: 2 copper layers, 95.2 x 48.3 mm, 9 parts, among them J1 Conn_NodeMCU_30pin_left, J2 Conn_NodeMCU_30pin_right, J3 Conn_NodeMCU_38pin_left, J4 Conn_NodeMCU_38pin_right, J5 Conn_Piezzo (aktiv/passiv), J6 Conn_LCD, SW1 SW_Meldung_bestätigen

Commit message: Layout-Datei zum ätzen für Dieter erzeugt
Parts:
- moved R1 6.73 mm to (140.8, 83.3)
- moved J6 6.73 mm to (126.1, 85.1)
- moved D1 6.73 mm to (138.3, 67.1)
- moved J5 6.73 mm to (126.1, 68.6)
- moved SW1 6.73 mm to (138.3, 61.0)
Routing:
- net +5V: track 150.8 -> 104.5 mm
- net Net-(J2-Pin_12): track 134.5 -> 107.7 mm
- net GND: track 145.8 -> 130.4 mm
- net Net-(J2-Pin_8): track 64.9 -> 79.5 mm
- net Net-(J2-Pin_11): track 58.9 -> 51.7 mm
- net Net-(J2-Pin_2): track 61.1 -> 54.3 mm
- net Net-(J2-Pin_5): track 70.5 -> 64.0 mm
- added copper zone on B.Cu, net (none)
Other:
- board size 95.2 x 48.3 mm -> 82.6 x 42.4 mm
- board text added: "42,42mm"
- board text added: "82,55mm"
- board text added: "Wenn dieser Text lesbar ist, ist der Druck gespiegelt"
- board text removed: "ca 48mm"
- board text removed: "ca. 95mm"
