File: KiCAD/NewsBox_V1/NewsBox.kicad_sch (KiCad schematic)
At the start: 9 parts, among them J1 Conn_NodeMCU_30pin_left, J2 Conn_NodeMCU_30pin_right, J3 Conn_NodeMCU_38pin_left, J4 Conn_NodeMCU_38pin_right, J5 Conn_Piezzo (aktiv/passiv), J6 Conn_LCD, SW1 SW_Meldung_bestätigen

Commit message: Layout-Datei zum ätzen für Dieter erzeugt
Other:
- title: (none) -> NewsBox Projekt
Changed lines of the file:
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@@
 	(generator_version "8.0")
 	(paper "A4")
+	(title_block
+		(title "NewsBox Projekt")
+		(date "2024-03-06")
+		(rev "1.0")
+	)
 	(junction
 		(at 134.62 101.6)
